Commit message: Refactor: Use base.stl for bot visual and collision
Co-authored-by: suhail17mohammad <suhail17mohammad@gmail.com>

File: hb_description/models/holonomic_bot/hb_bot.xacro (robot description, xacro)
@@ -91,5 +91,5 @@
             <origin xyz="0 0 0" rpy="0 0 0" />
             <geometry>
-                <mesh filename="file://$(find hb_description)/models/holonomic_bot/meshes/bot.dae"/>
+                <mesh filename="file://$(find hb_description)/models/holonomic_bot/meshes/base.stl"/>
             </geometry>
         </visual>
@@ -97,5 +97,5 @@
             <origin xyz="0 0 0.026" rpy="0 0 0" />
             <geometry>
-                <mesh filename="file://$(find hb_description)/models/holonomic_bot/meshes/bot.dae"/>
+                <mesh filename="file://$(find hb_description)/models/holonomic_bot/meshes/base.stl"/>
             </geometry>
         </collision>
